File: schtest/schtest/schtest.kicad_pcb (KiCad board)
At the start: 4 copper layers, 8 parts, among them P1 RZM001P02T2L, P2 RZM001P02T2L, P3 RZM001P02T2L

Commit message: Update design
Parts:
- added D1: LED, cnhardware:LED_0402_1005Metric_COMPACT, F.Cu at (157.9, 74.4)
- added R3: 1k, cnhardware:R_0402_1005Metric_COMPACT, F.Cu at (156.9, 74.4)
- N1, N2, N3: footprint Package_TO_SOT_SMD:SOT-723 -> cnhardware:SOT-723-COMPACT
- P1, P2, P3: footprint Package_TO_SOT_SMD:SOT-723 -> cnhardware:SOT-723-COMPACTP
- R1, R2: footprint Resistor_SMD:R_0402_1005Metric -> cnhardware:R_0402_1005Metric_COMPACT
- moved R1 0.90 mm to (157.4, 75.7)
- moved R2 0.86 mm to (157.3, 76.6)
- moved P1 0.15 mm to (155.7, 74.5)
- moved N1 0.14 mm to (155.7, 76.2)
- moved P2 0.14 mm to (159.1, 74.5)
- moved N2 0.12 mm to (159.1, 76.2)
Routing:
- net B0S: track 6.68 -> 5.02 mm
- net VDD: track 1.29 -> 2.68 mm
- net Net-(D1-K): track 0.00 -> 0.91 mm
- net B0Q: track 6.06 -> 5.49 mm
- net B0NQ: track 1.98 -> 2.51 mm
Other:
- board outline added: 12 x 10 mm
