File: schtest/schtest/schtest.kicad_sch (KiCad schematic)
At the start: 6 parts, among them P1 RZM001P02T2L, P2 RZM001P02T2L

Commit message: Cleanup schematic
Connections:
- net B0NQ: now also P1.3 (D); no longer P1.2 (S)
- net B0Q: now also P2.3 (D); no longer P2.2 (S)
- net VDD: now also P1.2 (S), P2.2 (S); no longer P1.3 (D), P2.3 (D)
Other:
- moved on the sheet: P1, R1, R2

Commit message: Bump designs
Parts:
- added N3: 2SK3541, Package_TO_SOT_SMD:SOT-723, symbol Device:Q_NMOS_GSD
- added P3: RZM001P02T2L, Package_TO_SOT_SMD:SOT-723, symbol Device:Q_PMOS_GSD
Connections:
- net B0Q: now also N3.1 (G), P3.1 (G)
- net GND: now also N3.2 (S)
- net VDD: now also P3.2 (S)
- new net: N3.3 (D), P3.3 (D)
Other:
- moved on the sheet: R1, R2

Commit message: Update design
Parts:
- added D1: LED, cnhardware:LED_0402_1005Metric_COMPACT, symbol Device:LED
- added R3: 1k, cnhardware:R_0402_1005Metric_COMPACT, symbol Device:R
- N1, N2, N3: footprint Package_TO_SOT_SMD:SOT-723 -> cnhardware:SOT-723-COMPACT
- P1, P2, P3: footprint Package_TO_SOT_SMD:SOT-723 -> cnhardware:SOT-723-COMPACTP
- R1, R2: footprint Resistor_SMD:R_0402_1005Metric -> cnhardware:R_0402_1005Metric_COMPACT
Connections:
- net B0NQ: now also R3.2
- net VDD: now also D1.2 (A)
- new net: D1.1 (K), R3.1
Changed lines of the file:
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@@
+	)
+	(junction
+		(at 29.21 35.56)
+		(diameter 0)
+		(color 0 0 0 0)
 	)
 	(junction
@@
 	(wire
 		(pts
-			(xy 46.99 45.72) (xy 53.34 45.72)
+			(xy 48.26 45.72) (xy 53.34 45.72)
+		)
+		(stroke
+			(width 0)
+			(type default)
+		)
+	)
+	(wire
+		(pts
+			(xy 21.59 45.72) (xy 21.59 44.45)
 		)
 		(stroke
@@
 	(wire
 		(pts
+			(xy 21.59 35.56) (xy 21.59 36.83)
+		)
+		(stroke
+			(width 0)
+			(type default)
+		)
+	)
+	(wire
+		(pts
 			(xy 38.1 46.99) (xy 38.1 45.72)
 		)
@@
 	(wire
 		(pts
-			(xy 46.99 39.37) (xy 46.99 45.72)
+			(xy 48.26 39.37) (xy 48.26 45.72)
 		)
 		(stroke
@@
 	(wire
 		(pts
+			(xy 21.59 45.72) (xy 29.21 45.72)
+		)
+		(stroke
+			(width 0)
+			(type default)
+		)
+	)
+	(wire
+		(pts
 			(xy 36.83 40.64) (xy 36.83 50.8)
 		)
@@
 	(wire
 		(pts
-			(xy 44.45 39.37) (xy 46.99 39.37)
+			(xy 44.45 39.37) (xy 48.26 39.37)
 		)
 		(stroke
@@
 			)
 		)
-		(property "Footprint" "Package_TO_SOT_SMD:SOT-723"
+		(property "Footprint" "cnhardware:SOT-723-COMPACTP"
 			(at 55.88 43.18 0)
 			(effects
@@
 		(dnp no)
 		(property "Reference" "P1"
-			(at 34.544 44.704 0)
+			(at 34.798 44.45 0)
 			(effects
 				(font
@@
 			)
 		)
-		(property "Footprint" "Package_TO_SOT_SMD:SOT-723"
+		(property "Footprint" "cnhardware:SOT-723-COMPACTP"
 			(at 26.67 43.18 0)
 			(effects
@@
 			)
 		)
-		(property "Footprint" "Package_TO_SOT_SMD:SOT-723"
+		(property "Footprint" "cnhardware:SOT-723-COMPACTP"
 			(at 77.47 43.18 0)
 			(effects
@@
 			)
 		)
-		(property "Footprint" "Package_TO_SOT_SMD:SOT-723"
+		(property "Footprint" "cnhardware:SOT-723-COMPACT"
 			(at 77.47 48.26 0)
 			(effects
@@
 		(dnp no)
 		(property "Reference" "N1"
-			(at 34.544 46.736 0)
+			(at 34.798 46.99 0)
 			(effects
 				(font
@@
 			)
 		)
-		(property "Footprint" "Package_TO_SOT_SMD:SOT-723"
+		(property "Footprint" "cnhardware:SOT-723-COMPACT"
 			(at 26.67 48.26 0)
 			(effects
@@
 				(path "/65a3ee60-5d53-43a0-a9e7-55cfb05b77d7"
 					(reference "N1")
+					(unit 1)
+				)
+			)
+		)
+	)
+	(symbol
+		(lib_id "Device:R")
+		(at 21.59 40.64 0)
+		(unit 1)
+		(exclude_from_sim no)
+		(in_bom yes)
+		(on_board yes)
+		(dnp no)
+		(property "Reference" "R3"
+			(at 23.876 40.64 0)
+			(effects
+				(font
+					(size 1.27 1.27)
+				)
+			)
+		)
+		(property "Value" "1k"
+			(at 21.59 40.386 90)
+			(effects
+				(font
+					(size 1.27 1.27)
+				)
+			)
+		)
+		(property "Footprint" "cnhardware:R_0402_1005Metric_COMPACT"
+			(at 19.812 40.64 90)
+			(effects
+				(font
+					(size 1.27 1.27)
+				)
+				(hide yes)
+			)
+		)
+		(property "Datasheet" "~"
+			(at 21.59 40.64 0)
+			(effects
+				(font
+					(size 1.27 1.27)
+				)
+				(hide yes)
+			)
+		)
+		(property "Description" "Resistor"
+			(at 21.59 40.64 0)
+			(effects
+				(font
+					(size 1.27 1.27)
+				)
+				(hide yes)
+			)
+		)
+		(property "LCSC" "C11702"
+			(at 21.59 40.64 90)
+			(effects
+				(font
+					(size 1.27 1.27)
+				)
+				(hide yes)
+			)
+		)
+		(pin "2"
+		)
+		(pin "1"
+		)
+		(instances
+			(project "schtest"
+				(path "/65a3ee60-5d53-43a0-a9e7-55cfb05b77d7"
+					(reference "R3")
+					(unit 1)
+				)
+			)
+		)
+	)
+	(symbol
+		(lib_id "Device:LED")
+		(at 25.4 35.56 0)
+		(unit 1)
+		(exclude_from_sim no)
+		(in_bom yes)
+		(on_board yes)
+		(dnp no)
+		(property "Reference" "D1"
+			(at 26.924 37.846 0)
+			(effects
+				(font
+					(size 1.27 1.27)
+				)
+				(justify right)
+			)
+		)
+		(property "Value" "LED"
+			(at 21.59 38.354 90)
+			(effects
+				(font
+					(size 1.27 1.27)
+				)
+				(justify right)
+				(hide yes)
+			)
+		)
+		(property "Footprint" "cnhardware:LED_0402_1005Metric_COMPACT"
+			(at 25.4 35.56 0)
+			(effects
+				(font
+					(size 1.27 1.27)
+				)
+				(hide yes)
+			)
+		)
+		(property "Datasheet" "~"
+			(at 25.4 35.56 0)
+			(effects
+				(font
+					(size 1.27 1.27)
+				)
+				(hide yes)
+			)
+		)
+		(property "Description" "Light emitting diode"
+			(at 25.4 35.56 0)
+			(effects
+				(font
+					(size 1.27 1.27)
+				)
+				(hide yes)
+			)
+		)
+		(property "LCSC" "C965793"
+			(at 25.4 35.56 90)
+			(effects
+				(font
+					(size 1.27 1.27)
+				)
+				(hide yes)
+			)
+		)
+		(property "Sim.Device" "D"
+			(at 25.4 35.56 0)
+			(effects
+				(font
+					(size 1.27 1.27)
+				)
+				(hide yes)
+			)
+		)
+		(property "Sim.Pins" "1=A 2=K"
+			(at 25.4 35.56 0)
+			(effects
+				(font
+					(size 1.27 1.27)
+				)
+				(hide yes)
+			)
+		)
+		(pin "1"
+		)
+		(pin "2"
+		)
+		(instances
+			(project "schtest"
+				(path "/65a3ee60-5d53-43a0-a9e7-55cfb05b77d7"
+					(reference "D1")
 					(unit 1)
 				)
@@
 		(dnp no)
 		(property "Reference" "N2"
-			(at 47.752 47.244 0)
+			(at 47.498 47.498 0)
 			(effects
 				(font
@@
 			)
 		)
-		(property "Footprint" "Package_TO_SOT_SMD:SOT-723"
+		(property "Footprint" "cnhardware:SOT-723-COMPACT"
 			(at 55.88 48.26 0)
 			(effects
@@
 			)
 		)
-		(property "Footprint" "Resistor_SMD:R_0402_1005Metric"
+		(property "Footprint" "cnhardware:R_0402_1005Metric_COMPACT"
 			(at 40.64 37.592 90)
 			(effects
@@
 			)
 		)
-		(property "Footprint" "Resistor_SMD:R_0402_1005Metric"
+		(property "Footprint" "cnhardware:R_0402_1005Metric_COMPACT"
 			(at 41.91 48.768 90)
 			(effects
