File: hwtest/hwtest.kicad_sch (KiCad schematic)
At the start: 299 parts, among them P1 RZM001P02T2L, P10 BSS84KNC, P11 BSS84KNC, P12 BSS84KNC, P13 BSS84KNC, P14 RZM001P02T2L, P15 RZM001P02T2L, P16 RZM001P02T2L, P17 BSS84KNC, P18 BSS84KNC, P19 BSS84KNC, P2 RZM001P02T2L, P20 RZM001P02T2L, P21 RZM001P02T2L, P22 RZM001P02T2L, P23 RZM001P02T2L, P24 RZM001P02T2L, P25 RZM001P02T2L, P26 RZM001P02T2L, P27 RZM001P02T2L, P28 BSS84KNC, P29 BSS84KNC, P3 RZM001P02T2L, P30 RZM001P02T2L, P31 RZM001P02T2L, P32 RZM001P02T2L, P33 RZM001P02T2L, P34 RZM001P02T2L, P35 RZM001P02T2L, P36 RZM001P02T2L, P37 RZM001P02T2L, P38 RZM001P02T2L, P39 RZM001P02T2L, P4 RZM001P02T2L, P40 RZM001P02T2L, P41 RZM001P02T2L, P42 RZM001P02T2L, P43 RZM001P02T2L, P44 RZM001P02T2L, P45 RZM001P02T2L, P46 RZM001P02T2L, P47 RZM001P02T2L, P48 RZM001P02T2L, P49 RZM001P02T2L, P5 RZM001P02T2L, P50 RZM001P02T2L, P51 RZM001P02T2L, P52 RZM001P02T2L, P53 RZM001P02T2L, P54 RZM001P02T2L, P55 RZM001P02T2L, P56 RZM001P02T2L, P57 RZM001P02T2L, P6 RZM001P02T2L, P7 RZM001P02T2L, P8 RZM001P02T2L, P9 BSS84KNC

Commit message: Tweak design.
Parts:
- added D19: LED, cnhardware:LED_0402_1005Metric_COMPACT, symbol Device:LED
- added N58, N59, N60, N61, N62, N63: 2SK3541, cnhardware:SOT-723-COMPACT, symbol Device:Q_NMOS_GSD
- added P58, P59, P60, P61, P62, P63: RZM001P02T2L, cnhardware:SOT-723-COMPACTP, symbol Device:Q_PMOS_GSD
- added R45: 1k, cnhardware:R_0402_1005Metric_COMPACT, symbol Device:R
- added TP124: XOR2A, cnhardware:TPTHRU, symbol Connector:TestPoint
- added TP125: XOR2B, cnhardware:TPTHRU, symbol Connector:TestPoint
- added TP126: XOR2O, cnhardware:TPTHRU, symbol Connector:TestPoint
Connections:
- net GND: now also N60.2 (S), N61.2 (S), N62.2 (S), N63.2 (S), R45.2
- net VDD: now also P58.2 (S), P59.2 (S), P62.2 (S), P63.2 (S)
- new net: N59.1 (G), N62.1 (G), P61.1 (G), P62.1 (G), TP124.1
- new net: N61.1 (G), N63.1 (G), P60.1 (G), P63.1 (G), TP125.1
- new net: N60.1 (G), N63.3 (D), P59.1 (G), P63.3 (D)
- new net: P58.3 (D), P59.3 (D), P60.2 (S), P61.2 (S)
- new net: D19.2 (A), N58.3 (D), N59.3 (D), P60.3 (D), P61.3 (D), TP126.1
- new net: N58.1 (G), N62.3 (D), P58.1 (G), P62.3 (D)
- new net: N59.2 (S), N61.3 (D)
- new net: D19.1 (K), R45.1
- new net: N58.2 (S), N60.3 (D)
Other:
- moved on the sheet: D13, D14, D15, D16, D17, D18, N28, N29, N30, N31, N32, N33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

Commit message: bump for order version
Parts:
- added R46, R47: 1k, cnhardware:R_0402_1005Metric_COMPACT, symbol Device:R
- added TP127: VCCXOR2, cnhardware:TPTHRU, symbol Connector:TestPoint
- added TP128: GNDXOR2, cnhardware:TPTHRU, symbol Connector:TestPoint
Connections:
- net GND: now also R46.2, R47.2, TP128.1
- net VDD: now also TP127.1
- net at N59.1 (G), N62.1 (G), P61.1 (G)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: now also R47.1
- net at N61.1 (G), N63.1 (G), P60.1 (G)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: now also R46.1
Other:
- note added: "N: RDS(ON)= 5Ω@VGS=10V, ID=200mA, 15pF CISS, 10pF COSS, VGSth = 1V (2SK3541) $0.0126 / C42402303 N: RDS(ON)= 3Ω@VGS=10V, ID= , 40pF CISS, 30pF COSS, VGSth = 1.3V (2N7002) $0.0097 P: RDS(ON)= 5Ω@VGS=10V, ID=130mA, 30pF CISS, 10pF COSS, VGSth =-1.3V (BSS84KT7) $0.0152 P: RDS(ON)=3.8Ω@VGS=10V, ID=100mA, 15pF CISS, 4pF COSS, VGSth =-0.6V (RZM001P02T2L) $0.0197 / **C308762** ... 1006 N: RDS(ON)=2.8Ω@V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"
- note removed: "N: RDS(ON)= 5Ω@VGS=10V, ID=200mA, 15pF CISS, 10pF COSS, VGSth = 1V (2SK3541) $0.0126 / C42402303 N: RDS(ON)= 3Ω@VGS=10V, ID= , 40pF CISS, 30pF COSS, VGSth = 1.3V (2N7002) $0.0097 P: RDS(ON)= 5Ω@VGS=10V, ID=130mA, 30pF CISS, 10pF COSS, VGSth =-1.3V (BSS84KT7) $0.0152 P: RDS(ON)=3.8Ω@VGS=10V, ID=100mA, 15pF CISS, 4pF COSS, VGSth =-0.6V (RZM001P02T2L) $0.0197 / C308762 ... 1006 N: RDS(ON)=2.8Ω@VGS=1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"
- moved on the sheet: D19, N58, N59, N60, N61, N62, N63, P58, P59, P60, P61, P62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

Commit message: Tweak test
Parts:
- added D20, D21: LED, cnhardware:LED_0402_1005Metric_COMPACT, symbol Device:LED
- added N64, N65, N66, N67, N68, N69, N70, N71, N72, N73, N74, N75, N76, N77: 2SK3541, cnhardware:DFN1006-3-NCH, symbol Device:Q_NMOS_GSD
- added P64, P65, P66, P67, P68, P69, P70, P71, P72, P73, P74, P75, P76, P77: RZM001P02T2L, cnhardware:DFN1006-3-PCH, symbol Device:Q_PMOS_GSD
- added R48, R49, R50, R51, R52: 1k, cnhardware:R_0402_1005Metric_COMPACT, symbol Device:R
- added TP129: FACi, cnhardware:TPTHRU, symbol Connector:TestPoint
- added TP130: FAB, cnhardware:TPTHRU, symbol Connector:TestPoint
- added TP131: FAA, cnhardware:TPTHRU, symbol Connector:TestPoint
- added TP132: FACO, cnhardware:TPTHRU, symbol Connector:TestPoint
- added TP133: FASO, cnhardware:TPTHRU, symbol Connector:TestPoint
- added TP134: VCCFA, cnhardware:TPTHRU, symbol Connector:TestPoint
- added TP135: GNDFA, cnhardware:TPTHRU, symbol Connector:TestPoint
- N10, N11, N12, N13, N17, N18, N19, N28, N29, N9: LCSC C3283163 -> C240200
- P10, P11, P12, P13, P17, P18, P19, P28, P29, P9: LCSC C41355123 -> C443620
Connections:
- net GND: now also N64.2 (S), N66.2 (S), N67.2 (S), N69.2 (S), N72.2 (S), N73.2 (S), N75.2 (S), N76.2 (S), N77.2 (S), R48.2, R49.2, R50.2, R51.2, R52.2, TP135.1
- net VDD: now also P64.2 (S), P67.2 (S), P68.2 (S), P70.2 (S), P72.2 (S), P76.2 (S), P77.2 (S), TP134.1
- new net: N73.3 (D), N74.2 (S), N75.3 (D), N77.3 (D)
- new net: P70.3 (D), P71.2 (S), P72.3 (D), P73.2 (S), P76.3 (D)
- new net: P73.3 (D), P74.2 (S)
- new net: P74.3 (D), P75.2 (S)
- new net: N70.3 (D), N74.3 (D), N76.1 (G), P71.3 (D), P75.3 (D), P77.1 (G)
- new net: N64.3 (D), N65.2 (S), N66.3 (D)
- new net: P64.3 (D), P65.2 (S), P68.3 (D), P69.2 (S)
- new net: D20.1 (K), R51.1
- new net: N68.2 (S), N69.3 (D)
- new net: P65.3 (D), P66.2 (S)
- new net: N70.2 (S), N71.3 (D)
- new net: D21.1 (K), R52.1
- new net: N71.2 (S), N72.3 (D)
- new net COUTs: D20.2 (A), N67.3 (D), P67.3 (D), TP132.1
- new net FAAs: N66.1 (G), N68.1 (G), N70.1 (G), N73.1 (G), P64.1 (G), P66.1 (G), P72.1 (G), P73.1 (G), R50.1, TP131.1
- new net FABs: N64.1 (G), N69.1 (G), N71.1 (G), N75.1 (G), P65.1 (G), P68.1 (G), P75.1 (G), P76.1 (G), R49.1, TP130.1
- new net FACis: N65.1 (G), N72.1 (G), N77.1 (G), P69.1 (G), P70.1 (G), P74.1 (G), R48.1, TP129.1
- new net SOUTs: D21.2 (A), N76.3 (D), P77.3 (D), TP133.1
- new net Xs: N65.3 (D), N67.1 (G), N68.3 (D), N74.1 (G), P66.3 (D), P67.1 (G), P69.3 (D), P71.1 (G)
Other:
- note added: "DISCUSS: I think we should not use SOT-883 (1006 size) 1. Harder to route (can't go under chip) 2. Can't probe chips. 3. Can't mess up rotation"
- moved on the sheet: D19, D7, D8, D9, N22, N23, N24, N25, N28, N29, N58, N59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
