File: sim4/kicad/kicad.kicad_sch (KiCad schematic)
At the start: 15 parts, among them P4 RZM001P02T2L, P5 RZM001P02T2L, P6 RZM001P02T2L, P7 RZM001P02T2L, P8 RZM001P02T2L

Commit message: Coming laong
Parts:
- renumbered D2 to LED1, N4 to N1, N5 to N2, N6 to N3, N7 to N4, N8 to N5, P4 to P1, P5 to P2, P6 to P3, P7 to P4, P8 to P5, R4 to R1, TP2 to TP1, TP1 to TP2, TP4 to TP3
Changed lines of the file:
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@@
 		(on_board yes)
 		(dnp no)
-		(property "Reference" "N6"
+		(property "Reference" "N3"
 			(at 59.182 34.544 0)
 			(effects
@@
 			(project "kicad"
 				(path "/d386f80f-1709-42ec-8243-5d17ab4d0026"
-					(reference "N6")
+					(reference "N3")
 					(unit 1)
 				)
@@
 		(on_board yes)
 		(dnp no)
-		(property "Reference" "#PWR011"
+		(property "Reference" "#PWR09"
 			(at 74.93 26.67 0)
 			(effects
@@
 			(project "kicad"
 				(path "/d386f80f-1709-42ec-8243-5d17ab4d0026"
-					(reference "#PWR011")
+					(reference "#PWR09")
 					(unit 1)
 				)
@@
 		(on_board yes)
 		(dnp no)
-		(property "Reference" "N4"
+		(property "Reference" "N1"
 			(at 38.862 34.544 0)
 			(effects
@@
 			(project "kicad"
 				(path "/d386f80f-1709-42ec-8243-5d17ab4d0026"
-					(reference "N4")
+					(reference "N1")
 					(unit 1)
 				)
@@
 		(on_board yes)
 		(dnp no)
-		(property "Reference" "N7"
+		(property "Reference" "N4"
 			(at 69.342 34.544 0)
 			(effects
@@
 			(project "kicad"
 				(path "/d386f80f-1709-42ec-8243-5d17ab4d0026"
-					(reference "N7")
+					(reference "N4")
 					(unit 1)
 				)
@@
 		(dnp no)
 		(fields_autoplaced yes)
-		(property "Reference" "TP4"
+		(property "Reference" "TP3"
 			(at 82.55 45.7199 90)
 			(effects
@@
 			)
 		)
-		(property "Sim.Device" "SPICE"
+		(property "Sim.Device" "TP"
 			(at 77.47 46.99 0)
 			(effects
@@
 			)
 		)
-		(property "Sim.Params" "type=TP_"
+		(property "Sim.Params" "TP"
 			(at 77.47 46.99 0)
 			(effects
@@
 			(project "kicad"
 				(path "/d386f80f-1709-42ec-8243-5d17ab4d0026"
-					(reference "TP4")
+					(reference "TP3")
 					(unit 1)
 				)
@@
 		(on_board yes)
 		(dnp no)
-		(property "Reference" "P6"
+		(property "Reference" "P3"
 			(at 58.166 24.638 0)
 			(effects
@@
 			(project "kicad"
 				(path "/d386f80f-1709-42ec-8243-5d17ab4d0026"
-					(reference "P6")
+					(reference "P3")
 					(unit 1)
 				)
@@
 		(on_board yes)
 		(dnp no)
-		(property "Reference" "#PWR015"
+		(property "Reference" "#PWR013"
 			(at 92.71 33.02 0)
 			(effects
@@
 			(project "kicad"
 				(path "/d386f80f-1709-42ec-8243-5d17ab4d0026"
-					(reference "#PWR015")
+					(reference "#PWR013")
 					(unit 1)
 				)
@@
 		(on_board yes)
 		(dnp no)
-		(property "Reference" "#PWR018"
+		(property "Reference" "#PWR01"
 			(at 29.21 33.02 0)
 			(effects
@@
 			(project "kicad"
 				(path "/d386f80f-1709-42ec-8243-5d17ab4d0026"
-					(reference "#PWR018")
+					(reference "#PWR01")
 					(unit 1)
 				)
@@
 		(on_board yes)
 		(dnp no)
-		(property "Reference" "#PWR09"
+		(property "Reference" "#PWR07"
 			(at 64.77 26.67 0)
 			(effects
@@
 			(project "kicad"
 				(path "/d386f80f-1709-42ec-8243-5d17ab4d0026"
-					(reference "#PWR09")
+					(reference "#PWR07")
 					(unit 1)
 				)
@@
 		(on_board yes)
 		(dnp no)
-		(property "Reference" "D2"
+		(property "Reference" "LED1"
 			(at 94.996 31.496 0)
 			(effects
@@
 			)
 		)
-		(property "Sim.Device" "D"
+		(property "Sim.Device" "LED"
 			(at 92.71 33.02 0)
 			(effects
@@
 			(project "kicad"
 				(path "/d386f80f-1709-42ec-8243-5d17ab4d0026"
-					(reference "D2")
+					(reference "LED1")
 					(unit 1)
 				)
@@
 		(on_board yes)
 		(dnp no)
-		(property "Reference" "P4"
+		(property "Reference" "P1"
 			(at 37.846 24.638 0)
 			(effects
@@
 			(project "kicad"
 				(path "/d386f80f-1709-42ec-8243-5d17ab4d0026"
-					(reference "P4")
+					(reference "P1")
 					(unit 1)
 				)
@@
 		(dnp no)
 		(fields_autoplaced yes)
-		(property "Reference" "TP1"
+		(property "Reference" "TP2"
 			(at 27.9399 34.29 90)
 			(effects
@@
 			)
 		)
-		(property "Sim.Device" "SPICE"
+		(property "Sim.Device" "TP"
 			(at 29.21 39.37 0)
 			(effects
@@
 			)
 		)
-		(property "Sim.Params" "type=TP_"
+		(property "Sim.Params" "TP"
 			(at 29.21 39.37 0)
 			(effects
@@
 			(project "kicad"
 				(path "/d386f80f-1709-42ec-8243-5d17ab4d0026"
-					(reference "TP1")
+					(reference "TP2")
 					(unit 1)
 				)
@@
 		(on_board yes)
 		(dnp no)
-		(property "Reference" "#PWR010"
+		(property "Reference" "#PWR08"
 			(at 64.77 49.53 0)
 			(effects
@@
 			(project "kicad"
 				(path "/d386f80f-1709-42ec-8243-5d17ab4d0026"
-					(reference "#PWR010")
+					(reference "#PWR08")
 					(unit 1)
 				)
@@
 		(on_board yes)
 		(dnp no)
-		(property "Reference" "#PWR07"
+		(property "Reference" "#PWR05"
 			(at 54.61 26.67 0)
 			(effects
@@
 			(project "kicad"
 				(path "/d386f80f-1709-42ec-8243-5d17ab4d0026"
-					(reference "#PWR07")
+					(reference "#PWR05")
 					(unit 1)
 				)
@@
 		(on_board yes)
 		(dnp no)
-		(property "Reference" "#PWR012"
+		(property "Reference" "#PWR010"
 			(at 74.93 49.53 0)
 			(effects
@@
 			(project "kicad"
 				(path "/d386f80f-1709-42ec-8243-5d17ab4d0026"
-					(reference "#PWR012")
+					(reference "#PWR010")
 					(unit 1)
 				)
@@
 		(on_board yes)
 		(dnp no)
-		(property "Reference" "#PWR05"
+		(property "Reference" "#PWR03"
 			(at 44.45 26.67 0)
 			(effects
@@
 			(project "kicad"
 				(path "/d386f80f-1709-42ec-8243-5d17ab4d0026"
-					(reference "#PWR05")
+					(reference "#PWR03")
 					(unit 1)
 				)
@@
 		(on_board yes)
 		(dnp no)
-		(property "Reference" "P8"
+		(property "Reference" "P5"
 			(at 78.486 24.638 0)
 			(effects
@@
 			(project "kicad"
 				(path "/d386f80f-1709-42ec-8243-5d17ab4d0026"
-					(reference "P8")
+					(reference "P5")
 					(unit 1)
 				)
@@
 		(on_board yes)
 		(dnp no)
-		(property "Reference" "#PWR08"
+		(property "Reference" "#PWR06"
 			(at 54.61 49.53 0)
 			(effects
@@
 			(project "kicad"
 				(path "/d386f80f-1709-42ec-8243-5d17ab4d0026"
-					(reference "#PWR08")
+					(reference "#PWR06")
 					(unit 1)
 				)
@@
 		(on_board yes)
 		(dnp no)
-		(property "Reference" "N8"
+		(property "Reference" "N5"
 			(at 79.502 34.544 0)
 			(effects
@@
 			(project "kicad"
 				(path "/d386f80f-1709-42ec-8243-5d17ab4d0026"
-					(reference "N8")
+					(reference "N5")
 					(unit 1)
 				)
@@
 		(dnp no)
 		(fields_autoplaced yes)
-		(property "Reference" "TP2"
+		(property "Reference" "TP1"
 			(at 27.9399 21.59 90)
 			(effects
@@
 			)
 		)
-		(property "Sim.Device" "SPICE"
+		(property "Sim.Device" "TP"
 			(at 29.21 26.67 0)
 			(effects
@@
 			)
 		)
-		(property "Sim.Params" "type=TP_"
+		(property "Sim.Params" "TP"
 			(at 29.21 26.67 0)
 			(effects
@@
 			(project "kicad"
 				(path "/d386f80f-1709-42ec-8243-5d17ab4d0026"
-					(reference "TP2")
+					(reference "TP1")
 					(unit 1)
 				)
@@
 		(on_board yes)
 		(dnp no)
-		(property "Reference" "#PWR013"
+		(property "Reference" "#PWR011"
 			(at 85.09 26.67 0)
 			(effects
@@
 			(project "kicad"
 				(path "/d386f80f-1709-42ec-8243-5d17ab4d0026"
-					(reference "#PWR013")
+					(reference "#PWR011")
 					(unit 1)
 				)
@@
 		(on_board yes)
 		(dnp no)
-		(property "Reference" "#PWR014"
+		(property "Reference" "#PWR012"
 			(at 85.09 49.53 0)
 			(effects
@@
 			(project "kicad"
 				(path "/d386f80f-1709-42ec-8243-5d17ab4d0026"
-					(reference "#PWR014")
+					(reference "#PWR012")
 					(unit 1)
 				)
@@
 		(on_board yes)
 		(dnp no)
-		(property "Reference" "P5"
+		(property "Reference" "P2"
 			(at 48.006 24.638 0)
 			(effects
@@
 			(project "kicad"
 				(path "/d386f80f-1709-42ec-8243-5d17ab4d0026"
-					(reference "P5")
+					(reference "P2")
 					(unit 1)
 				)
@@
 		(on_board yes)
 		(dnp no)
-		(property "Reference" "#PWR019"
+		(property "Reference" "#PWR02"
 			(at 29.21 35.56 0)
 			(effects
@@
 			(project "kicad"
 				(path "/d386f80f-1709-42ec-8243-5d17ab4d0026"
-					(reference "#PWR019")
+					(reference "#PWR02")
 					(unit 1)
 				)
@@
 		(on_board yes)
 		(dnp no)
-		(property "Reference" "#PWR06"
+		(property "Reference" "#PWR04"
 			(at 44.45 49.53 0)
 			(effects
@@
 			(project "kicad"
 				(path "/d386f80f-1709-42ec-8243-5d17ab4d0026"
-					(reference "#PWR06")
+					(reference "#PWR04")
 					(unit 1)
 				)
@@
 		(on_board yes)
 		(dnp no)
-		(property "Reference" "P7"
+		(property "Reference" "P4"
 			(at 68.326 24.638 0)
 			(effects
@@
 			(project "kicad"
 				(path "/d386f80f-1709-42ec-8243-5d17ab4d0026"
-					(reference "P7")
+					(reference "P4")
 					(unit 1)
 				)
@@
 		(on_board yes)
 		(dnp no)
-		(property "Reference" "R4"
+		(property "Reference" "R1"
 			(at 94.996 40.64 0)
 			(effects
@@
 			(project "kicad"
 				(path "/d386f80f-1709-42ec-8243-5d17ab4d0026"
-					(reference "R4")
+					(reference "R1")
 					(unit 1)
 				)
@@
 		(on_board yes)
 		(dnp no)
-		(property "Reference" "N5"
+		(property "Reference" "N2"
 			(at 49.022 34.544 0)
 			(effects
@@
 			(project "kicad"
 				(path "/d386f80f-1709-42ec-8243-5d17ab4d0026"
-					(reference "N5")
-					(unit 1)
-				)
+					(reference "N2")
+					(unit 1)
+				)
