File: kicad/kicad.kicad_sch (KiCad schematic)
At the start: 15 parts, among them P1 RZM001P02T2L, P2 RZM001P02T2L, P3 RZM001P02T2L, P4 RZM001P02T2L, P5 RZM001P02T2L

Commit message: Update showing functional sim
Parts:
- added N10, N11, N12, N13, N14, N15, N16, N17, N18, N19, N20, N21, N22, N23, N24, N25, N26, N6, N7, N8, N9: 2SK3541, cnhardware:SOT-723-COMPACT, symbol Device:Q_NMOS_GSD
- added P10, P11, P12, P13, P14, P15, P16, P17, P18, P19, P20, P21, P22, P23, P24, P25, P26, P6, P7, P8, P9: RZM001P02T2L, cnhardware:SOT-723-COMPACTP, symbol Device:Q_PMOS_GSD
- added R10, R2, R3, R4, R5: 1, cnhardware:R_0402_1005Metric_COMPACT, symbol Device:R
Connections:
- net GND: now also N11.2 (S), N13.2 (S), N14.2 (S), N16.2 (S), N18.2 (S), N20.2 (S), N22.2 (S), N23.2 (S), N24.2 (S), N25.2 (S), N26.2 (S), N6.2 (S), N7.2 (S), N8.2 (S), N9.2 (S)
- net MM1: now also N2.3 (D), P2.3 (D), N6.1 (G), P6.1 (G); no longer N4.3 (D), N5.1 (G), P4.3 (D), P5.1 (G), TP3.1
- net MM2: now also N6.3 (D), N9.1 (G), P6.3 (D), P9.1 (G); no longer N3.3 (D), N4.1 (G), P3.3 (D), P4.1 (G)
- net MM3: now also N7.1 (G), N9.3 (D), P7.1 (G), P9.3 (D); no longer N2.3 (D), N3.1 (G), P2.3 (D), P3.1 (G)
- net MM4: now also N7.3 (D), N8.1 (G), P7.3 (D), P8.1 (G); no longer N1.3 (D), N2.1 (G), P1.3 (D), P2.1 (G)
- net MONITOR: now also R4.1, R5.1
- net VDD: now also P10.2 (S), P11.2 (S), P12.2 (S), P13.2 (S), P14.2 (S), P16.2 (S), P18.2 (S), P19.2 (S), P21.2 (S), P23.2 (S), P24.2 (S), P25.2 (S), P26.2 (S), P6.2 (S), P7.2 (S), P8.2 (S), P9.2 (S)
- new net: N19.2 (S), N20.3 (D)
- new net: P19.3 (D), P20.2 (S)
- new net: N14.3 (D), P14.3 (D), R3.1
- new net: N12.2 (S), N13.3 (D)
- new net: P21.3 (D), P22.2 (S)
- new net: N21.2 (S), N22.3 (D)
- new net: N10.2 (S), N11.3 (D)
- new net DOUT: R10.2
- new net MIDTEST: N17.2 (S), N18.3 (D)
- new net MIDTEST2: P15.2 (S), P16.3 (D)
- new net MIDTEST3: N15.2 (S), N16.3 (D)
- new net MIDTEST4: P17.2 (S), P18.3 (D)
- new net MM0: N1.3 (D), N2.1 (G), P1.3 (D), P2.1 (G)
- new net MM5: N3.1 (G), N8.3 (D), P3.1 (G), P8.3 (D)
- new net MM6: N3.3 (D), N4.1 (G), P3.3 (D), P4.1 (G)
- new net MM7: N4.3 (D), N5.1 (G), P4.3 (D), P5.1 (G), TP3.1
- new net NAND01: N12.3 (D), N20.1 (G), N25.1 (G), P12.3 (D), P13.3 (D), P21.1 (G), P26.1 (G)
- new net NAND0O: N10.3 (D), N15.1 (G), N24.1 (G), P10.3 (D), P11.3 (D), P16.1 (G), P23.1 (G)
- new net NANDA0: N10.1 (G), P10.1 (G), R2.2
- new net NANDA1: N12.1 (G), P12.1 (G), R3.2
- new net NANDB0: N11.1 (G), P11.1 (G), R4.2
- new net NANDB1: N13.1 (G), P13.1 (G), R5.2
- new net XORA1: N15.3 (D), N17.3 (D), N19.1 (G), N23.1 (G), P15.3 (D), P17.3 (D), P19.1 (G), P25.1 (G)
- new net XORB0: N14.1 (G), N16.1 (G), N19.3 (D), N21.3 (D), N26.1 (G), P14.1 (G), P18.1 (G), P20.3 (D), P22.3 (D), P24.1 (G), R10.1, R2.1
- new net XORnA0: N17.1 (G), N24.3 (D), P17.1 (G), P23.3 (D)
- new net XORnA1: N21.1 (G), N23.3 (D), P22.1 (G), P25.3 (D)
- new net XORnB0: N18.1 (G), N26.3 (D), P15.1 (G), P24.3 (D)
- new net XORnB1: N22.1 (G), N25.3 (D), P20.1 (G), P26.3 (D)
Other:
- note added: "reattach"
- moved on the sheet: LED1, N1, N2, N3, N4, N5, P1, P2, P3, P4, P5, R1

Commit message: Add more tests
Parts:
- removed R10, R2, R3, R4, R5: 1, cnhardware:R_0402_1005Metric_COMPACT, symbol Device:R
- removed TP3: ROON, cnhardware:TPTHRU, symbol Connector:TestPoint
- added N27, N28, N29, N30, N31: 2SK3541, cnhardware:SOT-723-COMPACT, symbol Device:Q_NMOS_GSD
- added P27, P28, P29, P30, P31: RZM001P02T2L, cnhardware:SOT-723-COMPACTP, symbol Device:Q_PMOS_GSD
- added TP4: nXOR, cnhardware:TPTHRU, symbol Connector:TestPoint
- added TP5, TP6, TP7: TP, cnhardware:TPTHRU, symbol Connector:TestPoint
Connections:
- net NANDA0 is gone; now on net DOUT: N10.1 (G), P10.1 (G)
- net NANDA1 is gone; now on net BUFFERED_DIV2: N12.1 (G), P12.1 (G)
- net NANDB0 is gone; now on net MONITOR: N11.1 (G), P11.1 (G)
- net NANDB1 is gone; now on net MONITOR: N13.1 (G), P13.1 (G)
- net XORB0 is gone; now on net DOUT: N14.1 (G), N16.1 (G), N19.3 (D), N21.3 (D), N26.1 (G), P14.1 (G), P18.1 (G), P20.3 (D), P22.3 (D), P24.1 (G)
- net GND: now also N28.2 (S), N29.2 (S), N30.2 (S), N31.2 (S)
- net MONITOR: now also N29.1 (G), P29.1 (G)
- net VDD: now also P27.2 (S), P28.2 (S), P29.2 (S), P31.2 (S)
- net BUFFERED_DIV2: now reaches N14.3 (D), P14.3 (D)
- net BUFFERED_DIV2: now also N27.1 (G), N31.1 (G), P27.1 (G), P31.1 (G), TP4.1
- new net: N27.2 (S), N28.3 (D)
- new net: P30.2 (S), P31.3 (D)
- new net BUFFERED_CLK: N28.1 (G), N29.3 (D), N30.1 (G), P28.1 (G), P29.3 (D), P30.1 (G), TP6.1
- new net NANDTESTOUT: N27.3 (D), P27.3 (D), P28.3 (D), TP5.1
- new net NORTESTOUT: N30.3 (D), N31.3 (D), P30.3 (D), TP7.1

Commit message: More wacky circuits
Parts:
- added N32, N34: 2SK3541, cnhardware:SOT-723-COMPACT, symbol Device:Q_NMOS_GSD
- added P32, P33: RZM001P02T2L, cnhardware:SOT-723-COMPACTP, symbol Device:Q_PMOS_GSD
- added R2: 100, cnhardware:R_0402_1005Metric_COMPACT, symbol Device:R
- added TP3: TP, cnhardware:TPTHRU, symbol Connector:TestPoint
Connections:
- net BUFFERED_CLK: now also N32.1 (G), N34.2 (S), P33.1 (G)
- net BUFFERED_DIV2: now also N32.2 (S), N34.1 (G), P32.1 (G)
- net VDD: now also P32.2 (S), R2.1
- new net: P32.3 (D), P33.2 (S)
- new net XORTESTOUT: N32.3 (D), N34.3 (D), P33.3 (D), R2.2, TP3.1
